File: KiCad_Files/Sensors.sch (KiCad schematic (older format))
At the start: 48 parts, among them IC1 MAX6682MUA+T, IC2 MAX6682MUA+T, IC3 MAX6682MUA+T, IC4 MMC5983MA, IC5 ZMOD4410AI3V, J4 53261-7002, J5 53261-7002, J6 53261-7002, U4 MPU-6050, U6 MPX5070GP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

Commit message: Revert "Add shapes3D folder"
This reverts commit 1c3042b7a1c052b8553a455bf3bd885d3494e48a.
Parts:
- C20, C21, C23, C24, C25, C26, C27, C28, C29, C30, C31, C32, C33, C34, C35, C36: symbol archive:Device_C_Small -> Device:C_Small
- IC1, IC2, IC3: symbol archive:SamacSys_Parts_MAX6682MUA+T -> SamacSys_Parts:MAX6682MUA+T
- IC4: symbol archive:SamacSys_Parts_MMC5983MA -> SamacSys_Parts:MMC5983MA
- IC5: symbol archive:SamacSys_Parts_ZMOD4410AI3V -> SamacSys_Parts:ZMOD4410AI3V
- J4, J5, J6: symbol archive:SamacSys_Parts_53261-7002 -> SamacSys_Parts:53261-7002
- JP2, JP3, JP4: symbol archive:Jumper_SolderJumper_3_Open -> Jumper:SolderJumper_3_Open
- R16, R17, R18, R19, R20, R21, R22, R24: symbol archive:Device_R_Small -> Device:R_Small
- TP1, TP2, TP3, TP4, TP5, TP6: symbol archive:Connector_TestPoint -> Connector:TestPoint
- U4: symbol archive:Sensor_Motion_MPU-6050 -> Sensor_Motion:MPU-6050
- U6: symbol archive:Zenith_Modified_Libraries_MPX5070GP -> Zenith_Modified_Libraries:MPX5070GP
- U7: symbol archive:Sensor_Humidity_HDC1080 -> Sensor_Humidity:HDC1080
- U8: symbol archive:dk_Pressure-Sensors-Transducers_MS560702BA03-50 -> dk_Pressure-Sensors-Transducers:MS560702BA03-50
- VR1, VR2, VR3: symbol archive:SamacSys_Parts_TC33X-2-204E -> SamacSys_Parts:TC33X-2-204E

Commit message: Add shapes3D folder
Now all 3D models for the components are stored in a single folder, thanks to the Archive Plugin from https://github.com/MitjaNemec/Kicad_action_plugins.git
Parts:
- C20, C21, C23, C24, C25, C26, C27, C28, C29, C30, C31, C32, C33, C34, C35, C36: symbol Device:C_Small -> archive:Device_C_Small
- IC1, IC2, IC3: symbol SamacSys_Parts:MAX6682MUA+T -> archive:SamacSys_Parts_MAX6682MUA+T
- IC4: symbol SamacSys_Parts:MMC5983MA -> archive:SamacSys_Parts_MMC5983MA
- IC5: symbol SamacSys_Parts:ZMOD4410AI3V -> archive:SamacSys_Parts_ZMOD4410AI3V
- J4, J5, J6: symbol SamacSys_Parts:53261-7002 -> archive:SamacSys_Parts_53261-7002
- JP2, JP3, JP4: symbol Jumper:SolderJumper_3_Open -> archive:Jumper_SolderJumper_3_Open
- R16, R17, R18, R19, R20, R21, R22, R24: symbol Device:R_Small -> archive:Device_R_Small
- TP1, TP2, TP3, TP4, TP5, TP6: symbol Connector:TestPoint -> archive:Connector_TestPoint
- U4: symbol Sensor_Motion:MPU-6050 -> archive:Sensor_Motion_MPU-6050
- U6: symbol Zenith_Modified_Libraries:MPX5070GP -> archive:Zenith_Modified_Libraries_MPX5070GP
- U7: symbol Sensor_Humidity:HDC1080 -> archive:Sensor_Humidity_HDC1080
- U8: symbol dk_Pressure-Sensors-Transducers:MS560702BA03-50 -> archive:dk_Pressure-Sensors-Transducers_MS560702BA03-50
- VR1, VR2, VR3: symbol SamacSys_Parts:TC33X-2-204E -> archive:SamacSys_Parts_TC33X-2-204E
