File: KiCad_Files/Varella v.2.0.sch (KiCad schematic (older format))
At the start: 28 parts, among them J1 ESQ-120-39-G-D, J2 Conn_01x12_Male, U1 STM32L476RGTx, Y1 32,768k

Commit message: Revert "Add shapes3D folder again"
This reverts commit 7987a310af828f940c17547aa6162ac2ebe2b018.
Parts:
- 16M1: symbol archive:Device_Crystal_GND24 -> Device:Crystal_GND24
- C1, C10, C2, C3, C4, C5, C6, C7, C8, C9: symbol archive:Device_C_Small -> Device:C_Small
- D1: symbol archive:Device_LED -> Device:LED
- J1: symbol archive:SamacSys_Parts_ESQ-120-39-G-D -> SamacSys_Parts:ESQ-120-39-G-D
- J2: symbol archive:Connector_Conn_01x12_Male -> Connector:Conn_01x12_Male
- JP1: symbol archive:Jumper_SolderJumper_3_Open -> Jumper:SolderJumper_3_Open
- R1, R10, R11, R12, R13, R14, R15, R2, R3, R4: symbol archive:Device_R_Small -> Device:R_Small
- S1: symbol archive:SamacSys_Parts_PTS636_SM43J_SMTR_LFS -> SamacSys_Parts:PTS636_SM43J_SMTR_LFS
- U1: symbol archive:MCU_ST_STM32L4_STM32L476RGTx -> MCU_ST_STM32L4:STM32L476RGTx
- Y1: symbol archive:Device_Crystal_Small -> Device:Crystal_Small
Changed lines of the file:
@@
 	8575 4950 8625 4950
 $Comp
-L archive:MCU_ST_STM32L4_STM32L476RGTx U1
+L MCU_ST_STM32L4:STM32L476RGTx U1
 U 1 1 613E7615
 P 4625 5025
@@
 $EndComp
 $Comp
-L archive:power_+3.3V #PWR0101
+L power:+3.3V #PWR0101
 U 1 1 613F407B
 P 4675 3025
@@
 $EndComp
 $Comp
-L archive:power_GND #PWR0102
+L power:GND #PWR0102
 U 1 1 613FAFB6
 P 4625 6975
@@
 Connection ~ 4525 6925
 $Comp
-L archive:Device_C_Small C2
+L Device:C_Small C2
 U 1 1 614028ED
 P 4150 2050
@@
 $EndComp
 $Comp
-L archive:Device_C_Small C7
+L Device:C_Small C7
 U 1 1 6140503B
 P 4500 2050
@@
 $EndComp
 $Comp
-L archive:Device_C_Small C8
+L Device:C_Small C8
 U 1 1 614053AC
 P 4850 2050
@@
 $EndComp
 $Comp
-L archive:Device_C_Small C9
+L Device:C_Small C9
 U 1 1 6140585E
 P 5200 2050
@@
 $EndComp
 $Comp
-L archive:Device_C_Small C1
+L Device:C_Small C1
 U 1 1 61405AA7
 P 3800 2050
@@
 	4150 2250 4500 2250
 $Comp
-L archive:power_+3.3V #PWR0103
+L power:+3.3V #PWR0103
 U 1 1 61419BE2
 P 3800 1750
@@
 Connection ~ 3800 1850
 $Comp
-L archive:power_GND #PWR0104
+L power:GND #PWR0104
 U 1 1 6141BB41
 P 3800 2350
@@
 Connection ~ 3800 2250
 $Comp
-L archive:Device_R_Small R2
+L Device:R_Small R2
 U 1 1 6143BD59
 P 1900 3600
@@
 	2050 3600 2000 3600
 $Comp
-L archive:Jumper_SolderJumper_3_Open JP1
+L Jumper:SolderJumper_3_Open JP1
 U 1 1 61440C39
 P 1600 3600
@@
 	1750 3600 1800 3600
 $Comp
-L archive:power_+3.3V #PWR0105
+L power:+3.3V #PWR0105
 U 1 1 614479C3
 P 1600 3350
@@
 	1600 3350 1600 3400
 $Comp
-L archive:power_GND #PWR0106
+L power:GND #PWR0106
 U 1 1 61449D67
 P 1600 3850
@@
 	1600 3850 1600 3800
 $Comp
-L archive:Device_Crystal_GND24 16M1
+L Device:Crystal_GND24 16M1
 U 1 1 61450713
 P 1800 4950
@@
 $EndComp
 $Comp
-L archive:power_GND #PWR0107
+L power:GND #PWR0107
 U 1 1 61459354
 P 2725 5000
@@
 $EndComp
 $Comp
-L archive:power_GND #PWR0108
+L power:GND #PWR0108
 U 1 1 61459C79
 P 1325 5350
@@
 	2725 4950 2725 5000
 $Comp
-L archive:Device_C_Small C3
+L Device:C_Small C3
 U 1 1 6145E6A2
 P 1575 4700
@@
 	1800 4700 1800 4800
 $Comp
-L archive:Device_C_Small C4
+L Device:C_Small C4
 U 1 1 61463D13
 P 1575 5200
@@
 	3925 4725 3875 4725
 $Comp
-L archive:power_GND #PWR0110
+L power:GND #PWR0110
 U 1 1 614A349D
 P 1325 6650
@@
 	1325 6650 1325 6500
 $Comp
-L archive:Device_C_Small C5
+L Device:C_Small C5
 U 1 1 614A34A7
 P 1500 6125
@@
 	1400 6125 1325 6125
 $Comp
-L archive:Device_C_Small C6
+L Device:C_Small C6
 U 1 1 614A34B2
 P 1500 6500
@@
 	3925 6525 3875 6525
 $Comp
-L archive:power_+3.3V #PWR0111
+L power:+3.3V #PWR0111
 U 1 1 614C675D
 P 9575 5750
@@
 	9750 5975 9750 5925
 $Comp
-L archive:power_GND #PWR0112
+L power:GND #PWR0112
 U 1 1 614D5240
 P 9850 5975
@@
 	10650 6075 10650 5925
 $Comp
-L archive:power_GND #PWR0113
+L power:GND #PWR0113
 U 1 1 6158BF67
 P 1650 2600
@@
 $EndComp
 $Comp
-L archive:Device_R_Small R1
+L Device:R_Small R1
 U 1 1 6158C250
 P 1650 1750
@@
 $EndComp
 $Comp
-L archive:power_+3.3V #PWR0114
+L power:+3.3V #PWR0114
 U 1 1 6158C7F3
 P 1650 1550
@@
 	1650 1850 1650 1950
 $Comp
-L archive:Device_C_Small C10
+L Device:C_Small C10
 U 1 1 6159AFC7
 P 1850 2250
@@
 	3875 4925 3925 4925
 $Comp
-L archive:Device_LED D1
+L Device:LED D1
 U 1 1 61487691
 P 2700 2150
@@
 $EndComp
 $Comp
-L archive:power_GND #PWR0109
+L power:GND #PWR0109
 U 1 1 6149B9C4
 P 2700 2350
@@
 	2700 2300 2700 2350
 $Comp
-L archive:Device_R_Small R4
+L Device:R_Small R4
 U 1 1 614B0FAC
 P 2700 1850
@@
 GND
 $Comp
-L archive:power_+5V #PWR0116
+L power:+5V #PWR0116
 U 1 1 61683899
 P 6125 1850
@@
 $EndComp
 $Comp
-L archive:power_+3.3V #PWR0117
+L power:+3.3V #PWR0117
 U 1 1 61683C81
 P 6350 1850
@@
 $EndComp
 $Comp
-L archive:power_GND #PWR0118
+L power:GND #PWR0118
 U 1 1 61684B6A
 P 6250 2200
@@
 	5375 4225 5325 4225
 $Comp
-L archive:Device_R_Small R3
+L Device:R_Small R3
 U 1 1 614BCB98
 P 2050 5200
@@
 	1600 6500 1700 6500
 $Comp
-L archive:Device_Crystal_Small Y1
+L Device:Crystal_Small Y1
 U 1 1 614DD45F
 P 1700 6300
@@
 GND
 $Comp
-L archive:SamacSys_Parts_ESQ-120-39-G-D J1
+L SamacSys_Parts:ESQ-120-39-G-D J1
 U 1 1 613C51C6
 P 7675 5550
@@
 	10100 4875 10200 4875
 $Comp
-L archive:SamacSys_Parts_PTS636_SM43J_SMTR_LFS S1
+L SamacSys_Parts:PTS636_SM43J_SMTR_LFS S1
 U 1 1 6235C882
 P 1200 2250
@@
 UART_RX
 $Comp
-L archive:Connector_Conn_01x12_Male J2
+L Connector:Conn_01x12_Male J2
 U 1 1 6246EB1E
 P 10250 5725
@@
 SDA_B
 $Comp
-L archive:Device_R_Small R15
+L Device:R_Small R15
 U 1 1 617A79D8
 P 8850 1350
@@
 SDA_INA
 $Comp
-L archive:Device_R_Small R14
+L Device:R_Small R14
 U 1 1 618A4738
 P 8650 1350
@@
 $EndComp
 $Comp
-L archive:Device_R_Small R13
+L Device:R_Small R13
 U 1 1 618B1274
 P 8450 1350
@@
 $EndComp
 $Comp
-L archive:Device_R_Small R12
+L Device:R_Small R12
 U 1 1 618B127B
 P 8250 1350
@@
 $EndComp
 $Comp
-L archive:Device_R_Small R11
+L Device:R_Small R11
 U 1 1 618BDB75
 P 8050 1350
@@
 $EndComp
 $Comp
-L archive:Device_R_Small R10
+L Device:R_Small R10
 U 1 1 618BDB7C
 P 7850 1350
@@
 $EndComp
 $Comp
-L archive:power_+3.3V #PWR0139
+L power:+3.3V #PWR0139
 U 1 1 61739EA9
 P 8350 1100

Commit message: Archive Schematic
Parts:
- 16M1: symbol Device:Crystal_GND24 -> archive:Device_Crystal_GND24
- C1, C10, C2, C3, C4, C5, C6, C7, C8, C9: symbol Device:C_Small -> archive:Device_C_Small
- D1: symbol Device:LED -> archive:Device_LED
- J1: symbol SamacSys_Parts:ESQ-120-39-G-D -> archive:SamacSys_Parts_ESQ-120-39-G-D
- J2: symbol Connector:Conn_01x12_Male -> archive:Connector_Conn_01x12_Male
- JP1: symbol Jumper:SolderJumper_3_Open -> archive:Jumper_SolderJumper_3_Open
- R1, R10, R11, R12, R13, R14, R15, R2, R3, R4: symbol Device:R_Small -> archive:Device_R_Small
- S1: symbol SamacSys_Parts:PTS636_SM43J_SMTR_LFS -> archive:SamacSys_Parts_PTS636_SM43J_SMTR_LFS
- U1: symbol MCU_ST_STM32L4:STM32L476RGTx -> archive:MCU_ST_STM32L4_STM32L476RGTx
- Y1: symbol Device:Crystal_Small -> archive:Device_Crystal_Small
Changed lines of the file:
@@
 	8575 4950 8625 4950
 $Comp
-L MCU_ST_STM32L4:STM32L476RGTx U1
+L archive:MCU_ST_STM32L4_STM32L476RGTx U1
 U 1 1 613E7615
 P 4625 5025
@@
 $EndComp
 $Comp
-L power:+3.3V #PWR0101
+L archive:power_+3.3V #PWR0101
 U 1 1 613F407B
 P 4675 3025
@@
 $EndComp
 $Comp
-L power:GND #PWR0102
+L archive:power_GND #PWR0102
 U 1 1 613FAFB6
 P 4625 6975
@@
 Connection ~ 4525 6925
 $Comp
-L Device:C_Small C2
+L archive:Device_C_Small C2
 U 1 1 614028ED
 P 4150 2050
@@
 $EndComp
 $Comp
-L Device:C_Small C7
+L archive:Device_C_Small C7
 U 1 1 6140503B
 P 4500 2050
@@
 $EndComp
 $Comp
-L Device:C_Small C8
+L archive:Device_C_Small C8
 U 1 1 614053AC
 P 4850 2050
@@
 $EndComp
 $Comp
-L Device:C_Small C9
+L archive:Device_C_Small C9
 U 1 1 6140585E
 P 5200 2050
@@
 $EndComp
 $Comp
-L Device:C_Small C1
+L archive:Device_C_Small C1
 U 1 1 61405AA7
 P 3800 2050
@@
 	4150 2250 4500 2250
 $Comp
-L power:+3.3V #PWR0103
+L archive:power_+3.3V #PWR0103
 U 1 1 61419BE2
 P 3800 1750
@@
 Connection ~ 3800 1850
 $Comp
-L power:GND #PWR0104
+L archive:power_GND #PWR0104
 U 1 1 6141BB41
 P 3800 2350
@@
 Connection ~ 3800 2250
 $Comp
-L Device:R_Small R2
+L archive:Device_R_Small R2
 U 1 1 6143BD59
 P 1900 3600
@@
 	2050 3600 2000 3600
 $Comp
-L Jumper:SolderJumper_3_Open JP1
+L archive:Jumper_SolderJumper_3_Open JP1
 U 1 1 61440C39
 P 1600 3600
@@
 	1750 3600 1800 3600
 $Comp
-L power:+3.3V #PWR0105
+L archive:power_+3.3V #PWR0105
 U 1 1 614479C3
 P 1600 3350
@@
 	1600 3350 1600 3400
 $Comp
-L power:GND #PWR0106
+L archive:power_GND #PWR0106
 U 1 1 61449D67
 P 1600 3850
@@
 	1600 3850 1600 3800
 $Comp
-L Device:Crystal_GND24 16M1
+L archive:Device_Crystal_GND24 16M1
 U 1 1 61450713
 P 1800 4950
@@
 $EndComp
 $Comp
-L power:GND #PWR0107
+L archive:power_GND #PWR0107
 U 1 1 61459354
 P 2725 5000
@@
 $EndComp
 $Comp
-L power:GND #PWR0108
+L archive:power_GND #PWR0108
 U 1 1 61459C79
 P 1325 5350
@@
 	2725 4950 2725 5000
 $Comp
-L Device:C_Small C3
+L archive:Device_C_Small C3
 U 1 1 6145E6A2
 P 1575 4700
@@
 	1800 4700 1800 4800
 $Comp
-L Device:C_Small C4
+L archive:Device_C_Small C4
 U 1 1 61463D13
 P 1575 5200
@@
 	3925 4725 3875 4725
 $Comp
-L power:GND #PWR0110
+L archive:power_GND #PWR0110
 U 1 1 614A349D
 P 1325 6650
@@
 	1325 6650 1325 6500
 $Comp
-L Device:C_Small C5
+L archive:Device_C_Small C5
 U 1 1 614A34A7
 P 1500 6125
@@
 	1400 6125 1325 6125
 $Comp
-L Device:C_Small C6
+L archive:Device_C_Small C6
 U 1 1 614A34B2
 P 1500 6500
@@
 	3925 6525 3875 6525
 $Comp
-L power:+3.3V #PWR0111
+L archive:power_+3.3V #PWR0111
 U 1 1 614C675D
 P 9575 5750
@@
 	9750 5975 9750 5925
 $Comp
-L power:GND #PWR0112
+L archive:power_GND #PWR0112
 U 1 1 614D5240
 P 9850 5975
@@
 	10650 6075 10650 5925
 $Comp
-L power:GND #PWR0113
+L archive:power_GND #PWR0113
 U 1 1 6158BF67
 P 1650 2600
@@
 $EndComp
 $Comp
-L Device:R_Small R1
+L archive:Device_R_Small R1
 U 1 1 6158C250
 P 1650 1750
@@
 $EndComp
 $Comp
-L power:+3.3V #PWR0114
+L archive:power_+3.3V #PWR0114
 U 1 1 6158C7F3
 P 1650 1550
@@
 	1650 1850 1650 1950
 $Comp
-L Device:C_Small C10
+L archive:Device_C_Small C10
 U 1 1 6159AFC7
 P 1850 2250
@@
 	3875 4925 3925 4925
 $Comp
-L Device:LED D1
+L archive:Device_LED D1
 U 1 1 61487691
 P 2700 2150
@@
 $EndComp
 $Comp
-L power:GND #PWR0109
+L archive:power_GND #PWR0109
 U 1 1 6149B9C4
 P 2700 2350
@@
 	2700 2300 2700 2350
 $Comp
-L Device:R_Small R4
+L archive:Device_R_Small R4
 U 1 1 614B0FAC
 P 2700 1850
@@
 GND
 $Comp
-L power:+5V #PWR0116
+L archive:power_+5V #PWR0116
 U 1 1 61683899
 P 6125 1850
@@
 $EndComp
 $Comp
-L power:+3.3V #PWR0117
+L archive:power_+3.3V #PWR0117
 U 1 1 61683C81
 P 6350 1850
@@
 $EndComp
 $Comp
-L power:GND #PWR0118
+L archive:power_GND #PWR0118
 U 1 1 61684B6A
 P 6250 2200
@@
 	5375 4225 5325 4225
 $Comp
-L Device:R_Small R3
+L archive:Device_R_Small R3
 U 1 1 614BCB98
 P 2050 5200
@@
 	1600 6500 1700 6500
 $Comp
-L Device:Crystal_Small Y1
+L archive:Device_Crystal_Small Y1
 U 1 1 614DD45F
 P 1700 6300
@@
 GND
 $Comp
-L SamacSys_Parts:ESQ-120-39-G-D J1
+L archive:SamacSys_Parts_ESQ-120-39-G-D J1
 U 1 1 613C51C6
 P 7675 5550
@@
 	10100 4875 10200 4875
 $Comp
-L SamacSys_Parts:PTS636_SM43J_SMTR_LFS S1
+L archive:SamacSys_Parts_PTS636_SM43J_SMTR_LFS S1
 U 1 1 6235C882
 P 1200 2250
@@
 UART_RX
 $Comp
-L Connector:Conn_01x12_Male J2
+L archive:Connector_Conn_01x12_Male J2
 U 1 1 6246EB1E
 P 10250 5725
@@
 SDA_B
 $Comp
-L Device:R_Small R15
+L archive:Device_R_Small R15
 U 1 1 617A79D8
 P 8850 1350
@@
 SDA_INA
 $Comp
-L Device:R_Small R14
+L archive:Device_R_Small R14
 U 1 1 618A4738
 P 8650 1350
@@
 $EndComp
 $Comp
-L Device:R_Small R13
+L archive:Device_R_Small R13
 U 1 1 618B1274
 P 8450 1350
@@
 $EndComp
 $Comp
-L Device:R_Small R12
+L archive:Device_R_Small R12
 U 1 1 618B127B
 P 8250 1350
@@
 $EndComp
 $Comp
-L Device:R_Small R11
+L archive:Device_R_Small R11
 U 1 1 618BDB75
 P 8050 1350
@@
 $EndComp
 $Comp
-L Device:R_Small R10
+L archive:Device_R_Small R10
 U 1 1 618BDB7C
 P 7850 1350
@@
 $EndComp
 $Comp
-L power:+3.3V #PWR0139
+L archive:power_+3.3V #PWR0139
 U 1 1 61739EA9
 P 8350 1100

Commit message: Add Traces to Stack Connector
Connects the Interrupts and PWM pins that come from the EPS boards through the Stack Connector to Varella's STM32.
Connections:
- net ZMOD_INT: now also U1.35 (PB14); no longer U1.36 (PB15)
- net EPS_ALRT1: now reaches J1.33
- net EPS_ALRT1: now also U1.42 (PA9)
- net EPS_CHRG: now reaches J1.34
- net EPS_CHRG: now also U1.58 (PB6)
- net EPS_THERM_PWM: now reaches J1.35
- net EPS_THERM_PWM: now also U1.56 (PB4)
- net EPS_FAULT: now reaches J1.37
- net EPS_FAULT: now also U1.50 (PA15)
- no-connect marks 36 -> 28
Other:
- moved on the sheet: J1
Changed lines of the file:
@@
 Comment4 ""
 $EndDescr
-Text GLabel 8625 3650 2    50   Input ~ 0
+Text GLabel 8675 3650 2    50   Input ~ 0
 GND
-Text GLabel 8625 3750 2    50   Input ~ 0
+Text GLabel 8675 3750 2    50   Input ~ 0
 GND
-Text GLabel 8625 4950 2    50   Input ~ 0
+Text GLabel 8675 4950 2    50   Input ~ 0
 BUS_RX1
-Text GLabel 8625 4450 2    50   Input ~ 0
+Text GLabel 8675 4450 2    50   Input ~ 0
 CAN_L
-Text GLabel 8625 4350 2    50   Input ~ 0
+Text GLabel 8675 4350 2    50   Input ~ 0
 CAN_H
-Text GLabel 8625 4150 2    50   Input ~ 0
+Text GLabel 8675 4150 2    50   Input ~ 0
 3V3
-Text GLabel 8625 4050 2    50   Input ~ 0
+Text GLabel 8675 4050 2    50   Input ~ 0
 5V
 Wire Wire Line
-	8575 3650 8625 3650
-Wire Wire Line
-	8575 3750 8625 3750
-Wire Wire Line
-	8575 4050 8625 4050
-Wire Wire Line
-	8575 4150 8625 4150
-Wire Wire Line
-	8575 4350 8625 4350
-Wire Wire Line
-	8575 4450 8625 4450
-Wire Wire Line
-	8575 4950 8625 4950
+	8625 3650 8675 3650
+Wire Wire Line
+	8625 3750 8675 3750
+Wire Wire Line
+	8625 4050 8675 4050
+Wire Wire Line
+	8625 4150 8675 4150
+Wire Wire Line
+	8625 4350 8675 4350
+Wire Wire Line
+	8625 4450 8675 4450
+Wire Wire Line
+	8625 4950 8675 4950
 $Comp
 L archive:MCU_ST_STM32L4_STM32L476RGTx U1
@@
 Wire Wire Line
 	5325 6525 5375 6525
-Wire Wire Line
-	5325 6625 5375 6625
 Wire Wire Line
 	5325 5125 5375 5125
@@
 STM32L476RGT6
 Wire Wire Line
-	7625 4950 7675 4950
-Wire Wire Line
-	7625 4550 7675 4550
-Wire Wire Line
-	7625 4450 7675 4450
-Wire Wire Line
-	7625 4150 7675 4150
-Wire Wire Line
-	7625 4050 7675 4050
-Wire Wire Line
-	7625 3750 7675 3750
-Wire Wire Line
-	7625 3650 7675 3650
-Text GLabel 7625 4950 0    50   Input ~ 0
+	7675 4950 7725 4950
+Wire Wire Line
+	7675 4550 7725 4550
+Wire Wire Line
+	7675 4450 7725 4450
+Wire Wire Line
+	7675 4150 7725 4150
+Wire Wire Line
+	7675 4050 7725 4050
+Wire Wire Line
+	7675 3750 7725 3750
+Wire Wire Line
+	7675 3650 7725 3650
+Text GLabel 7675 4950 0    50   Input ~ 0
 BUS_TX1
-Text GLabel 7625 4150 0    50   Input ~ 0
+Text GLabel 7675 4150 0    50   Input ~ 0
 3V3
-Text GLabel 7625 4050 0    50   Input ~ 0
+Text GLabel 7675 4050 0    50   Input ~ 0
 5V
-Text GLabel 7625 3750 0    50   Input ~ 0
+Text GLabel 7675 3750 0    50   Input ~ 0
 GND
-Text GLabel 7625 3650 0    50   Input ~ 0
+Text GLabel 7675 3650 0    50   Input ~ 0
 GND
 $Comp
 L archive:SamacSys_Parts_ESQ-120-39-G-D J1
 U 1 1 613C51C6
-P 7675 5550
-F 0 "J1" H 8125 3650 50  0000 C CNN
-F 1 "ESQ-120-39-G-D" H 8150 3475 50  0000 C CNN
-F 2 "SamacSys_Parts:ESQ-120-Y-X-D" H 8425 5650 50  0001 L CNN
-F 3 "http://suddendocs.samtec.com/prints/esq-1xx-xx-x-x-xxx-xx-x-xx-mkt.pdf" H 8425 5550 50  0001 L CNN
-F 4 "40 Position, Elevated Socket Strip, 0.100&quot; Pitch" H 8425 5450 50  0001 L CNN "Description"
-F 5 "" H 8425 5350 50  0001 L CNN "Height"
-F 6 "200-ESQ12039GD" H 8425 5250 50  0001 L CNN "Mouser Part Number"
-F 7 "https://www.mouser.co.uk/ProductDetail/Samtec/ESQ-120-39-G-D?qs=FESYatJ8odKQoQHulXlnvA%3D%3D" H 8425 5150 50  0001 L CNN "Mouser Price/Stock"
-F 8 "SAMTEC" H 8425 5050 50  0001 L CNN "Manufacturer_Name"
-F 9 "ESQ-120-39-G-D" H 8425 4950 50  0001 L CNN "Manufacturer_Part_Number"
-	1    7675 5550
+P 7725 5550
+F 0 "J1" H 8175 3650 50  0000 C CNN
+F 1 "ESQ-120-39-G-D" H 8200 3475 50  0000 C CNN
+F 2 "SamacSys_Parts:ESQ-120-Y-X-D" H 8475 5650 50  0001 L CNN
+F 3 "http://suddendocs.samtec.com/prints/esq-1xx-xx-x-x-xxx-xx-x-xx-mkt.pdf" H 8475 5550 50  0001 L CNN
+F 4 "40 Position, Elevated Socket Strip, 0.100&quot; Pitch" H 8475 5450 50  0001 L CNN "Description"
+F 5 "" H 8475 5350 50  0001 L CNN "Height"
+F 6 "200-ESQ12039GD" H 8475 5250 50  0001 L CNN "Mouser Part Number"
+F 7 "https://www.mouser.co.uk/ProductDetail/Samtec/ESQ-120-39-G-D?qs=FESYatJ8odKQoQHulXlnvA%3D%3D" H 8475 5150 50  0001 L CNN "Mouser Price/Stock"
+F 8 "SAMTEC" H 8475 5050 50  0001 L CNN "Manufacturer_Name"
+F 9 "ESQ-120-39-G-D" H 8475 4950 50  0001 L CNN "Manufacturer_Part_Number"
+	1    7725 5550
 	1    0    0    1
 $EndComp
 NoConn ~ 10550 5925
-NoConn ~ 7675 3950
-NoConn ~ 7675 4250
-NoConn ~ 7675 4350
-NoConn ~ 8575 3950
-NoConn ~ 8575 4250
-NoConn ~ 8575 4550
-NoConn ~ 8575 4650
-NoConn ~ 8575 5050
-NoConn ~ 8575 5150
-NoConn ~ 8575 5250
-NoConn ~ 8575 5350
-NoConn ~ 8575 5450
-NoConn ~ 8575 5550
-NoConn ~ 7675 5550
-NoConn ~ 7675 5450
-NoConn ~ 7675 5350
-NoConn ~ 7675 5250
-NoConn ~ 7675 5150
-NoConn ~ 7675 5050
-NoConn ~ 7675 4650
+NoConn ~ 7725 3950
+NoConn ~ 7725 4250
+NoConn ~ 7725 4350
+NoConn ~ 8625 3950
+NoConn ~ 8625 4250
+NoConn ~ 8625 4550
+NoConn ~ 8625 4650
+NoConn ~ 8625 5050
+NoConn ~ 8625 5150
+NoConn ~ 8625 5350
+NoConn ~ 8625 5450
+NoConn ~ 8625 5550
+NoConn ~ 7725 5550
+NoConn ~ 7725 5150
+NoConn ~ 7725 5050
+NoConn ~ 7725 4650
 Text GLabel 10100 4575 0    50   Input ~ 0
 CAN_TX
@@
 Text GLabel 5375 4425 2    50   Input ~ 0
 MAX_3_NSS
-Text GLabel 7625 4550 0    50   Input ~ 0
+Text GLabel 7675 4550 0    50   Input ~ 0
 SCL_INA
-Text GLabel 7625 4450 0    50   Input ~ 0
+Text GLabel 7675 4450 0    50   Input ~ 0
 SDA_INA
-NoConn ~ 7675 4850
-NoConn ~ 8575 4850
-Text GLabel 8575 4750 2    50   Input ~ 0
+NoConn ~ 7725 4850
+NoConn ~ 8625 4850
+Text GLabel 8625 4750 2    50   Input ~ 0
 SCL_A
-Text GLabel 7675 4750 0    50   Input ~ 0
+Text GLabel 7725 4750 0    50   Input ~ 0
 SDA_A
 Text GLabel 3875 5125 0    50   Input ~ 0
@@
 Text GLabel 5375 5125 2    50   Input ~ 0
 MPX_VOUT
-NoConn ~ 5375 4325
-NoConn ~ 5375 4925
 NoConn ~ 5375 5225
-NoConn ~ 5375 5525
-NoConn ~ 5375 5725
 NoConn ~ 3875 5625
 NoConn ~ 3875 5825
-NoConn ~ 8575 3850
-NoConn ~ 7675 3850
+NoConn ~ 8625 3850
+NoConn ~ 7725 3850
 Text Notes 7075 6425 0    50   ~ 0
 MAX17205 I2C Address: 0x6C & 0x16\n(Connected to I2C_A on the stack bus )
@@
 Text GLabel 3875 5725 0    50   Input ~ 0
 ZMOD_RST
-Text GLabel 5375 6625 2    50   Input ~ 0
+Text GLabel 5375 6525 2    50   Input ~ 0
 ZMOD_INT
-NoConn ~ 5375 6525
+NoConn ~ 5325 6625
 NoConn ~ 3875 5525
 $Bitmap
@@
 EndData
 $EndBitmap
+Text GLabel 7725 5250 0    50   Input ~ 0
+EPS_ALRT1
+Text GLabel 7725 5350 0    50   Input ~ 0
+EPS_THERM_PWM
+Text GLabel 8625 5250 2    50   Input ~ 0
+EPS_CHRG
+Text GLabel 7725 5450 0    50   Input ~ 0
+EPS_FAULT
+Text GLabel 5375 5725 2    50   Input ~ 0
+EPS_CHRG
+Text GLabel 5375 5525 2    50   Input ~ 0
+EPS_THERM_PWM
+Text GLabel 5375 4925 2    50   Input ~ 0
+EPS_FAULT
+Text GLabel 5375 4325 2    50   Input ~ 0
+EPS_ALRT1
 $EndSCHEMATC
